File: boards/proto1_0/proto1_0.kicad_pcb (KiCad board)
At the start: 2 copper layers, 65 x 44 mm, 47 parts, among them J1 Conn_01x04, J2 Conn_ARM_JTAG_SWD_10, J3 Conn_01x01, Q1 SSM3J378R, SW1 2223-TS02-66-70-BK-160-LCR-D-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, SW2 2223-TS02-66-70-BK-160-LCR-D-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, U1 BT832, U2 ADS1230, Y1 32.768kHz

Commit message: Fix bad transistor pin assignment
The load cell power switch (Q1) used a PFET symbol that incorrectly
numbered its pins relative to the industry-standard for SOT-23 packages.
Use a more accurate symbol instead and fix the layout accordingly.

While a P1.1 board is not (yet) planned since this issue should be easy
to work around,, I've kept the footprint locations the same so that the
P1.0 stencil can be reused.
Connections:
- Q1 pad 1: /E+ -> Net-(Q1-G)
- Q1 pad 2: Net-(Q1-G) -> VCC
- Q1 pad 3: VCC -> /E+
Routing:
- net Net-(Q1-G): track 4.14 -> 7.43 mm
- net /E+: track 17.5 -> 19.7 mm
- net VCC: track 33.5 -> 32.2 mm
Other:
- board text added: "GND"
- board text added: "Hangman P1.1"
- board text removed: "Hangman P1.0"
Changed lines of the file:
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@@
     (property "Sheetname" "")
     (property "Sim.Device" "PMOS")
-    (property "Sim.Pins" "1=D 2=G 3=S")
+    (property "Sim.Pins" "1=G 2=S 3=D")
     (property "Sim.Type" "VDMOS")
-    (property "ki_description" "P-MOSFET transistor, drain/source/gate")
-    (property "ki_keywords" "transistor PMOS P-MOS P-MOSFET simulation")
+    (property "ki_description" "P-MOSFET transistor, gate/source/drain")
+    (property "ki_keywords" "transistor PMOS P-MOS P-MOSFET")
     (attr smd)
     (fp_text reference "Q1" (at -0.889 -2.794 -180) (layer "F.SilkS")
@@
       (stroke (width 0.1) (type solid)) (layer "F.Fab"))
     (pad "1" smd roundrect (at -0.9375 -0.95 270) (size 1.475 0.6) (layers "F.Cu" "F.Paste" "F.Mask") (roundrect_rratio 0.25)
-      (net 3 "/E+") (pinfunction "D") (pintype "passive"))
-    (pad "2" smd roundrect (at -0.9375 0.95 270) (size 1.475 0.6) (layers "F.Cu" "F.Paste" "F.Mask") (roundrect_rratio 0.25)
       (net 31 "Net-(Q1-G)") (pinfunction "G") (pintype "input"))
-    (pad "3" smd roundrect (at 0.9375 0 270) (size 1.475 0.6) (layers "F.Cu" "F.Paste" "F.Mask") (roundrect_rratio 0.25)
+    (pad "2" smd roundrect (at -0.9375 0.95 270) (size 1.475 0.6) (layers "F.Cu" "F.Paste" "F.Mask") (roundrect_rratio 0.25)
       (net 2 "VCC") (pinfunction "S") (pintype "passive"))
+    (pad "3" smd roundrect (at 0.9375 0 270) (size 1.475 0.6) (layers "F.Cu" "F.Paste" "F.Mask") (roundrect_rratio 0.25)
+      (net 3 "/E+") (pinfunction "D") (pintype "passive"))
     (model "${KICAD6_3DMODEL_DIR}/Package_TO_SOT_SMD.3dshapes/SOT-23.wrl"
       (offset (xyz 0 0 0))
@@
     (descr "SMD Crystal FC-135 https://support.epson.biz/td/api/doc_check.php?dl=brief_FC-135R_en.pdf")
     (tags "SMD SMT Crystal")
-    (property "Part number" " (FC31M2-32.768-N07LLDTL)")
+    (property "Part number" "SC32S-7PF20PPM")
     (property "Sheetfile" "proto1_0.kicad_sch")
     (property "Sheetname" "")
@@
   (gr_line (start 76.2 93.98) (end 76.2 81.915)
     (stroke (width 0.1) (type default)) (layer "Edge.Cuts"))
-  (gr_line (start 76.2 55.245) (end 76.2 49.9872)
-    (stroke (width 0.1) (type default)) (layer "Edge.Cuts"))
   (gr_line (start 141.2 49.9872) (end 141.2 93.98)
     (stroke (width 0.1) (type default)) (layer "Edge.Cuts"))
+  (gr_line (start 76.2 55.245) (end 76.2 49.9872)
+    (stroke (width 0.1) (type default)) (layer "Edge.Cuts"))
   (gr_line (start 100.33 82.55) (end 111.76 82.55)
     (stroke (width 0.1) (type default)) (layer "Edge.Cuts"))
@@
     (effects (font (size 0.762 0.762) (thickness 0.1524) bold) (justify left bottom))
   )
-  (gr_text "Hangman P1.0" (at 125.222 84.201) (layer "F.SilkS")
+  (gr_text "Hangman P1.1" (at 125.222 84.201) (layer "F.SilkS")
     (effects (font (size 1 1) (thickness 0.15)) (justify left bottom))
   )
@@
     (effects (font (size 0.762 0.762) (thickness 0.1524)) (justify left bottom))
   )
+  (gr_text "GND" (at 113.6142 82.0928) (layer "F.SilkS")
+    (effects (font (size 0.762 0.762) (thickness 0.1524) bold) (justify left bottom))
+  )
   (gr_text "~{VDDA_ON}" (at 104.267 57.658) (layer "F.SilkS")
     (effects (font (size 0.762 0.762) (thickness 0.1524) bold) (justify left bottom))
@@
   (segment (start 122.004 69.398) (end 121.793 69.609) (width 0.254) (layer "F.Cu") (net 2))
   (segment (start 123.6425 70.048) (end 124.531 70.048) (width 0.254) (layer "F.Cu") (net 2))
+  (segment (start 118.0846 59.7329) (end 118.0846 60.2996) (width 0.381) (layer "F.Cu") (net 2))
   (segment (start 120.2925 78.74) (end 120.2925 77.3195) (width 0.254) (layer "F.Cu") (net 2))
   (segment (start 127.254 71.058369) (end 127.254 71.689631) (width 0.254) (layer "F.Cu") (net 2))
@@
   (segment (start 127.700369 72.136) (end 129.2295 72.136) (width 0.254) (layer "F.Cu") (net 2))
   (segment (start 92.136 60.264) (end 92.136 59.182) (width 0.254) (layer "F.Cu") (net 2))
-  (segment (start 116.84 60.515) (end 119.9025 60.515) (width 0.254) (layer "F.Cu") (net 2))
-  (segment (start 119.9025 60.515) (end 120.015 60.6275) (width 0.254) (layer "F.Cu") (net 2))
+  (segment (start 119.065 58.7525) (end 118.0846 59.7329) (width 0.381) (layer "F.Cu") (net 2))
   (segment (start 123.6425 69.398) (end 123.6425 70.048) (width 0.254) (layer "F.Cu") (net 2))
   (segment (start 128.264369 70.048) (end 127.254 71.058369) (width 0.254) (layer "F.Cu") (net 2))
@@
   (segment (start 99.568 63.246) (end 99.568 63.373) (width 0.2032) (layer "B.Cu") (net 2))
   (segment (start 124.968 66.154) (end 124.968 67.818) (width 0.254) (layer "F.Cu") (net 3))
-  (segment (start 121.605 56.134) (end 120.965 56.774) (width 0.508) (layer "F.Cu") (net 3))
-  (segment (start 120.965 56.774) (end 120.965 58.7525) (width 0.508) (layer "F.Cu") (net 3))
+  (segment (start 121.605 56.6826) (end 122.428 57.5056) (width 0.508) (layer "F.Cu") (net 3))
+  (segment (start 124.6 62.0652) (end 124.6 64.7954) (width 0.508) (layer "F.Cu") (net 3))
+  (segment (start 122.428 59.8932) (end 121.8946 60.4266) (width 0.508) (layer "F.Cu") (net 3))
   (segment (start 121.605 54.202) (end 121.959 53.848) (width 0.254) (layer "F.Cu") (net 3))
   (segment (start 124.688 68.098) (end 123.6425 68.098) (width 0.254) (layer "F.Cu") (net 3))
   (segment (start 124.6 65.786) (end 124.968 66.154) (width 0.2032) (layer "F.Cu") (net 3))
+  (segment (start 120.015 60.6275) (end 121.6937 60.6275) (width 0.381) (layer "F.Cu") (net 3))
   (segment (start 124.968 67.818) (end 124.688 68.098) (width 0.254) (layer "F.Cu") (net 3))
-  (segment (start 124.6 62.3875) (end 120.965 58.7525) (width 0.2032) (layer "F.Cu") (net 3))
-  (segment (start 124.6 65.786) (end 124.6 62.3875) (width 0.2032) (layer "F.Cu") (net 3))
+  (segment (start 121.6937 60.6275) (end 121.8946 60.4266) (width 0.381) (layer "F.Cu") (net 3))
+  (segment (start 121.605 56.134) (end 121.605 56.6826) (width 0.508) (layer "F.Cu") (net 3))
+  (segment (start 122.428 57.5056) (end 122.428 59.8932) (width 0.508) (layer "F.Cu") (net 3))
   (segment (start 121.605 56.134) (end 121.605 54.202) (width 0.508) (layer "F.Cu") (net 3))
+  (segment (start 122.428 59.8932) (end 124.6 62.0652) (width 0.508) (layer "F.Cu") (net 3))
+  (segment (start 124.6 65.786) (end 124.6 64.7954) (width 0.2032) (layer "F.Cu") (net 3))
   (segment (start 83.91144 62.738) (end 83.439 62.26556) (width 0.2032) (layer "F.Cu") (net 4))
   (segment (start 87.63 57.195) (end 87.63 58.801) (width 0.2032) (layer "F.Cu") (net 4))
@@
   (segment (start 129.794 60.756499) (end 129.003 59.965499) (width 0.2) (layer "F.Cu") (net 27))
   (segment (start 129.003 59.965499) (end 129.003 57.604) (width 0.2) (layer "F.Cu") (net 27))
-  (segment (start 116.84 58.865) (end 118.9525 58.865) (width 0.2032) (layer "F.Cu") (net 31))
+  (segment (start 118.2248 57.4802) (end 116.84 58.865) (width 0.2032) (layer "F.Cu") (net 31))
   (segment (start 114.998 58.801) (end 116.776 58.801) (width 0.2032) (layer "F.Cu") (net 31))
   (segment (start 116.776 58.801) (end 116.84 58.865) (width 0.2032) (layer "F.Cu") (net 31))
-  (segment (start 118.9525 58.865) (end 119.065 58.7525) (width 0.2032) (layer "F.Cu") (net 31))
+  (segment (start 120.965 58.1762) (end 120.269 57.4802) (width 0.2032) (layer "F.Cu") (net 31))
+  (segment (start 120.269 57.4802) (end 118.2248 57.4802) (width 0.2032) (layer "F.Cu") (net 31))
+  (segment (start 120.965 58.7525) (end 120.965 58.1762) (width 0.2032) (layer "F.Cu") (net 31))
   (zone (net 2) (net_name "VCC") (layer "F.Cu") (hatch edge 0.5)
     (priority 2)
