File: boards/proto1_0/proto1_0.kicad_sch (KiCad schematic)
At the start: 47 parts, among them J1 Conn_01x04, J2 Conn_ARM_JTAG_SWD_10, J3 Conn_01x01, Q1 SSM3J378R, SW1 2223-TS02-66-70-BK-160-LCR-D-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, SW2 2223-TS02-66-70-BK-160-LCR-D-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, U1 BT832, U2 ADS1230, Y1 32.768kHz

Commit message: Fix bad transistor pin assignment
The load cell power switch (Q1) used a PFET symbol that incorrectly
numbered its pins relative to the industry-standard for SOT-23 packages.
Use a more accurate symbol instead and fix the layout accordingly.

While a P1.1 board is not (yet) planned since this issue should be easy
to work around,, I've kept the footprint locations the same so that the
P1.0 stencil can be reused.
Parts:
- Q1: symbol Simulation_SPICE:PMOS -> Device:Q_PMOS_GSD
- Y1: Part number (FC31M2-32.768-N07LLDTL) -> SC32S-7PF20PPM
Connections:
- net E+: now also Q1.3 (D); no longer Q1.1 (D)
- net VCC: now also Q1.2 (S); no longer Q1.3 (S)
- net at R7.2, R9.2: now also Q1.1 (G); no longer Q1.2 (G)
Other:
- note added: "Low-frequency crystal Load = (C1 + 4pF) / 2"
- note removed: "Low-frequency crystal"
Changed lines of the file:
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@@
 (kicad_sch (version 20230121) (generator eeschema)
   (paper "A4")
-  (junction (at 146.05 66.675) (diameter 0) (color 0 0 0 0)
-  )
   (junction (at 248.285 55.88) (diameter 0) (color 0 0 0 0)
   )
@@
   )
   (junction (at 62.865 118.745) (diameter 0) (color 0 0 0 0)
-  )
-  (junction (at 142.875 78.105) (diameter 0) (color 0 0 0 0)
   )
   (junction (at 127.635 182.88) (diameter 0) (color 0 0 0 0)
@@
     (stroke (width 0) (type default))
   )
-  (wire (pts (xy 146.05 76.2) (xy 146.05 78.105))
-    (stroke (width 0) (type default))
-  )
   (wire (pts (xy 67.945 74.93) (xy 67.945 71.755))
     (stroke (width 0) (type default))
@@
     (stroke (width 0) (type default))
   )
-  (wire (pts (xy 146.05 78.105) (xy 142.875 78.105))
-    (stroke (width 0) (type default))
-  )
   (wire (pts (xy 17.78 56.515) (xy 17.78 69.85))
     (stroke (width 0) (type default))
@@
     (stroke (width 0) (type default))
   )
-  (wire (pts (xy 132.715 66.675) (xy 146.05 66.675))
-    (stroke (width 0) (type default))
-  )
   (wire (pts (xy 135.89 88.265) (xy 135.89 91.44))
     (stroke (width 0) (type default))
@@
     (stroke (width 0) (type default))
   )
-  (wire (pts (xy 146.05 66.675) (xy 146.05 68.58))
-    (stroke (width 0) (type default))
-  )
   (wire (pts (xy 34.29 67.31) (xy 41.275 67.31))
     (stroke (width 0) (type default))
@@
     (stroke (width 0) (type default))
   )
-  (wire (pts (xy 146.05 66.675) (xy 149.86 66.675))
+  (wire (pts (xy 132.715 66.675) (xy 149.86 66.675))
     (stroke (width 0) (type default))
   )
@@
     (stroke (width 0) (type default))
   )
-  (wire (pts (xy 142.875 78.105) (xy 142.875 69.215))
-    (stroke (width 0) (type default))
-  )
   (wire (pts (xy 201.295 107.315) (xy 215.9 107.315))
     (stroke (width 0) (type default))
@@
     (stroke (width 0) (type default))
   )
-  (wire (pts (xy 142.875 91.44) (xy 142.875 78.105))
+  (wire (pts (xy 142.875 69.215) (xy 142.875 91.44))
     (stroke (width 0) (type default))
   )
@@
     (effects (font (size 1.27 1.27)) (justify left bottom))
   )
-  (text "Low-frequency crystal" (at 16.51 55.245 0)
+  (text "Low-frequency crystal\nLoad = (C1 + 4pF) / 2" (at 16.51 55.245 0)
     (effects (font (size 1.27 1.27)) (justify left bottom))
   )
@@
     )
   )
-  (symbol (lib_id "Simulation_SPICE:PMOS") (at 198.755 99.06 0) (mirror x) (unit 1)
+  (symbol (lib_id "Device:Q_PMOS_GSD") (at 198.755 99.06 0) (mirror x) (unit 1)
     (in_bom yes) (on_board yes) (dnp no) (fields_autoplaced)
     (property "Reference" "Q1" (at 204.47 97.79 0)
@@
       (effects (font (size 1.27 1.27)) hide)
     )
-    (property "Sim.Pins" "1=D 2=G 3=S" (at 198.755 83.82 0)
+    (property "Sim.Pins" "1=G 2=S 3=D" (at 198.755 83.82 0)
       (effects (font (size 1.27 1.27)) hide)
     )
@@
       (effects (font (size 1.27 1.27)) hide)
     )
-    (property "Part number" " (FC31M2-32.768-N07LLDTL)" (at 34.29 62.23 90)
-      (effects (font (size 1.27 1.27)) hide)
-    )
+    (property "Part number" "SC32S-7PF20PPM" (at 34.29 62.23 90)
+      (effects (font (size 1.27 1.27)) hide)
+    )

Commit message: Fix flipped PCB silkscreen
The white and green color labels for the load cell differential output
voltage pins were switched. There's no real functional effect since the
negative polarity would be fixed in calibration, but one can swap the
wires if desired.
Other:
- note added: "E+: Red E-: Black IN+: Green/Blue IN-: White Shield: Yellow"
- note removed: "E+: Red E-: Black IN-: White IN+: Green/Blue Shield: Yellow"
Changed lines of the file:
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@@
     (effects (font (size 1.27 1.27)) (justify left bottom))
   )
-  (text "E+: Red\nE-: Black\nIN-: White\nIN+: Green/Blue\nShield: Yellow"
+  (text "E+: Red\nE-: Black\nIN+: Green/Blue\nIN-: White\nShield: Yellow"
     (at 14.605 119.38 0)
     (effects (font (size 1.27 1.27)) (justify left bottom))
